File: transmitter/pcb/transmitter.kicad_sch (KiCad schematic)
At the start: 14 parts, among them U1 AMS1117-3.3, U2 MOUDLE-SEEEDUINO-XIAO-ESP32C3

Commit message: added 9v battery holder footprint and symbol
Parts:
- added U3: 9Vbattery, 9v_battery:9v_battery, symbol 9v:9Vbattery
Connections:
- net +9V: now also U3.2 (+)
- net GND: now also U3.1 (-)
- no-connect marks 9 -> 10
Changed lines of the file:
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@@
   (junction (at 99.06 170.18) (diameter 0) (color 0 0 0 0)
   )
-  (no_connect (at 142.24 121.92))
   (no_connect (at 74.93 81.28))
   (no_connect (at 171.45 86.36))
   (no_connect (at 74.93 86.36))
   (no_connect (at 121.92 172.72))
+  (no_connect (at 171.45 101.6))
   (no_connect (at 121.92 109.22))
+  (no_connect (at 171.45 97.79))
   (no_connect (at 73.66 128.27))
   (no_connect (at 92.71 35.56))
@@
     (pin "2")
   )
+  (symbol (lib_id "power:+9V") (at 237.49 114.3 0) (unit 1)
+    (in_bom yes) (on_board yes)
+    (property "Reference" "#PWR0102" (id 0) (at 237.49 118.11 0)
+      (effects (font (size 1.27 1.27)) hide)
+    )
+    (property "Value" "+9V" (id 1) (at 237.871 109.9058 0))
+    (property "Footprint" "" (id 2) (at 237.49 114.3 0)
+      (effects (font (size 1.27 1.27)) hide)
+    )
+    (property "Datasheet" "" (id 3) (at 237.49 114.3 0)
+      (effects (font (size 1.27 1.27)) hide)
+    )
+    (pin "1")
+  )
   (symbol (lib_id "Device:LED") (at 68.58 166.37 90) (unit 1)
     (in_bom yes) (on_board yes)
@@
     )
     (pin "1")
+  )
+  (symbol (lib_id "9v:9Vbattery") (at 227.33 118.11 0) (unit 1)
+    (in_bom yes) (on_board yes) (fields_autoplaced)
+    (property "Reference" "U3" (id 0) (at 242.57 139.6999 0)
+      (effects (font (size 1.27 1.27)) (justify left))
+    )
+    (property "Value" "9Vbattery" (id 1) (at 242.57 142.2399 0)
+      (effects (font (size 1.27 1.27)) (justify left))
+    )
+    (property "Footprint" "9v_battery:9v_battery" (id 2) (at 227.33 118.11 0)
+      (effects (font (size 1.27 1.27)) hide)
+    )
+    (property "Datasheet" "" (id 3) (at 227.33 118.11 0)
+      (effects (font (size 1.27 1.27)) hide)
+    )
+    (pin "1")
+    (pin "2")
   )
   (symbol (lib_id "SEEEDUINO-XIAO-ESP32C3:MOUDLE-SEEEDUINO-XIAO-ESP32C3") (at 147.32 97.79 0) (unit 1)
@@
     (pin "1")
   )
+  (symbol (lib_id "power:GND") (at 217.17 114.3 180) (unit 1)
+    (in_bom yes) (on_board yes)
+    (property "Reference" "#PWR0103" (id 0) (at 217.17 107.95 0)
+      (effects (font (size 1.27 1.27)) hide)
+    )
+    (property "Value" "GND" (id 1) (at 217.043 109.9058 0))
+    (property "Footprint" "" (id 2) (at 217.17 114.3 0)
+      (effects (font (size 1.27 1.27)) hide)
+    )
+    (property "Datasheet" "" (id 3) (at 217.17 114.3 0)
+      (effects (font (size 1.27 1.27)) hide)
+    )
+    (pin "1")
+  )
   (symbol (lib_id "power:GND") (at 53.34 181.61 0) (unit 1)
     (in_bom yes) (on_board yes)
@@
       (reference "#PWR0101") (unit 1) (value "GND") (footprint "")
     )
+    (path "/4add9cff-ae6c-494c-b447-b2edc764588e"
+      (reference "#PWR0102") (unit 1) (value "+9V") (footprint "")
+    )
+    (path "/7fcad4da-7c3b-4d88-ba59-b5a0ae398845"
+      (reference "#PWR0103") (unit 1) (value "GND") (footprint "")
+    )
     (path "/ad5ea85b-18ce-40c9-9cd4-e0ab3469cbfc"
       (reference "600ohm1") (unit 1) (value "R_US") (footprint "Resistor_SMD:R_0805_2012Metric_Pad1.20x1.40mm_HandSolder")
@@
       (reference "U2") (unit 1) (value "MOUDLE-SEEEDUINO-XIAO-ESP32C3") (footprint "xiao ESP32C3_PCB:MOUDLE14P-SMD-2.54-21X17.8MM")
     )
+    (path "/5ae1b3b4-e73a-4a98-9e35-508ba995514c"
+      (reference "U3") (unit 1) (value "9Vbattery") (footprint "9v_battery:9v_battery")
+    )
     (path "/dfaa4bc8-b037-4bd5-ad90-0f674345f5b8"
